File: Lutron Fountain.kicad_pcb (KiCad board)
At the start: 4 copper layers, 103 parts, among them J1 Barrel_Jack_MountingPin, Q1 BC547, Q10 BC547, Q11 BC547, Q12 BC547, Q13 BC547, Q14 BC547, Q15 BC547, Q16 BC547, Q17 BC547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

Commit message: finalized
Parts:
- removed D10, D11, D13, D15, D17, D18, D2, D21, D22, D25, D26, D29, D30, D33, D34, D35, D36, D4, D6, D8: RLED, LED_THT:LED_D5.0mm
- added J10: LED, TerminalBlock:TerminalBlock_MaiXu_MX126-5.0-02P_1x02_P5.00mm, F.Cu at (165.1, 106.8)
- added J11: LED, TerminalBlock:TerminalBlock_MaiXu_MX126-5.0-02P_1x02_P5.00mm, F.Cu at (177.8, 106.8)
- added J12: LED, TerminalBlock:TerminalBlock_MaiXu_MX126-5.0-02P_1x02_P5.00mm, F.Cu at (81.3, 111.7)
- added J13: LED, TerminalBlock:TerminalBlock_MaiXu_MX126-5.0-02P_1x02_P5.00mm, F.Cu at (68.6, 111.7)
- added J14: LED, TerminalBlock:TerminalBlock_MaiXu_MX126-5.0-02P_1x02_P5.00mm, F.Cu at (55.9, 111.7)
- added J15: LED, TerminalBlock:TerminalBlock_MaiXu_MX126-5.0-02P_1x02_P5.00mm, F.Cu at (43.2, 111.7)
- added J16: LED, TerminalBlock:TerminalBlock_MaiXu_MX126-5.0-02P_1x02_P5.00mm, F.Cu at (30.5, 111.8)
- added J17: LED, TerminalBlock:TerminalBlock_MaiXu_MX126-5.0-02P_1x02_P5.00mm, F.Cu at (81.3, 53.3)
- added J18: LED, TerminalBlock:TerminalBlock_MaiXu_MX126-5.0-02P_1x02_P5.00mm, F.Cu at (68.6, 53.3)
- added J19: LED, TerminalBlock:TerminalBlock_MaiXu_MX126-5.0-02P_1x02_P5.00mm, F.Cu at (55.9, 53.3)
- added J2: LED, TerminalBlock:TerminalBlock_MaiXu_MX126-5.0-02P_1x02_P5.00mm, F.Cu at (127.0, 48.3)
- added J20: LED, TerminalBlock:TerminalBlock_MaiXu_MX126-5.0-02P_1x02_P5.00mm, F.Cu at (43.2, 53.3)
- added J21: LED, TerminalBlock:TerminalBlock_MaiXu_MX126-5.0-02P_1x02_P5.00mm, F.Cu at (30.5, 53.3)
- added J3: LED, TerminalBlock:TerminalBlock_MaiXu_MX126-5.0-02P_1x02_P5.00mm, F.Cu at (139.7, 48.3)
- added J4: LED, TerminalBlock:TerminalBlock_MaiXu_MX126-5.0-02P_1x02_P5.00mm, F.Cu at (152.5, 48.3)
- added J5: LED, TerminalBlock:TerminalBlock_MaiXu_MX126-5.0-02P_1x02_P5.00mm, F.Cu at (165.1, 48.3)
- added J6: LED, TerminalBlock:TerminalBlock_MaiXu_MX126-5.0-02P_1x02_P5.00mm, F.Cu at (177.8, 48.3)
- added J7: LED, TerminalBlock:TerminalBlock_MaiXu_MX126-5.0-02P_1x02_P5.00mm, F.Cu at (127.0, 106.8)
- added J8: LED, TerminalBlock:TerminalBlock_MaiXu_MX126-5.0-02P_1x02_P5.00mm, F.Cu at (139.7, 106.8)
- added J9: LED, TerminalBlock:TerminalBlock_MaiXu_MX126-5.0-02P_1x02_P5.00mm, F.Cu at (152.4, 106.8)
- J1: value Barrel_Jack_MountingPin -> Power; footprint Connector_BarrelJack:BarrelJack_CUI_PJ-102AH_Horizontal -> TerminalBlock:TerminalBlock_MaiXu_MX126-5.0-02P_1x02_P5.00mm
- moved R12 7.62 mm to (127.0, 127.0)
- moved R14 7.62 mm to (139.7, 127.0)
- moved R16 7.62 mm to (152.4, 127.0)
- moved R18 7.62 mm to (165.1, 127.0)
- moved R20 7.62 mm to (177.8, 127.0)
- moved R23 7.62 mm to (81.3, 127.0)
- moved R27 7.62 mm to (68.6, 127.0)
- moved R31 7.62 mm to (55.9, 127.0)
- moved R35 7.62 mm to (43.2, 127.0)
- moved R39 7.62 mm to (30.5, 127.0)
- moved R10 6.35 mm to (177.8, 34.3)
- moved R2 6.35 mm to (127.0, 34.3)
- moved R24 6.35 mm to (81.3, 34.3)
- moved R28 6.35 mm to (68.6, 34.3)
- moved R32 6.35 mm to (55.9, 34.3)
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Connections:
- J1 pad 1: +5V -> GND
- J1 pad 2: GND -> +5V
Routing:
- net Net-(J16-Pin_1): track 0.00 -> 7.62 mm
- net Net-(J4-Pin_2): track 5.08 -> 7.73 mm
- net Net-(J9-Pin_1): track 5.08 -> 7.70 mm
- net Net-(J8-Pin_1): track 5.08 -> 7.70 mm
- net Net-(J7-Pin_1): track 5.08 -> 7.70 mm
- net Net-(J6-Pin_2): track 5.08 -> 7.70 mm
- net Net-(J5-Pin_2): track 5.08 -> 7.70 mm
- net Net-(J3-Pin_2): track 5.08 -> 7.70 mm
- net Net-(J21-Pin_1): track 5.08 -> 7.70 mm
- net Net-(J20-Pin_1): track 5.08 -> 7.70 mm
- net Net-(J2-Pin_2): track 5.08 -> 7.70 mm
- net Net-(J19-Pin_1): track 5.08 -> 7.70 mm
- net Net-(J18-Pin_1): track 5.08 -> 7.70 mm
- net Net-(J17-Pin_1): track 5.08 -> 7.70 mm
- net Net-(J16-Pin_2): track 5.08 -> 7.70 mm
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
Commit message: final
Other:
- board outline added: 172.7 x 104.1 mm
Changed lines of the file:
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@@
 		(tenting front back)
 		(pcbplotparams
-			(layerselection 0x00000000_00000000_55555555_5755f5ff)
+			(layerselection 0x00000000_00000000_55555555_575555ff)
 			(plot_on_all_layers_selection 0x00000000_00000000_00000000_00000000)
 			(disableapertmacros no)
@@
 			(outputformat 1)
 			(mirror no)
-			(drillshape 1)
+			(drillshape 0)
 			(scaleselection 1)
-			(outputdirectory "")
+			(outputdirectory "gerber")
 		)
 	)
@@
 		(layer "F.SilkS")
 	)
+	(gr_rect
+		(start 17.78 30.48)
+		(end 190.5 134.62)
+		(stroke
+			(width 0.05)
+			(type default)
+		)
+		(fill no)
+		(layer "Edge.Cuts")
+	)
 	(gr_text "Lutron Competition		Anna Tretiakova & Annalisa Emanuele		https://github.com/Shapitsa/Fountain-2026"
